Commit message: Kuka demo 03 - added poly-line trajectory and different configurations.

File: agimus_demo_03_mpc_dummy_traj_kuka/urdf/obstacles_none.xacro (robot description, xacro)
@@ -21,5 +21,5 @@
         </visual>
     <collision>
-      <origin xyz="0.6 0.0 0.15" />
+      <origin xyz="-0.5 0.0 0.15" />
       <geometry>
         <cylinder length="0.3" radius="0.1" />
@@ -28,5 +28,5 @@
      <!-- Note: these two are deleted in collision model update (robot_model.py)-->
      <collision>
-      <origin xyz="0.6 0.0 0.3" />
+      <origin xyz="-0.5 0.0 0.3" />
       <geometry>
         <sphere radius="0.1" />
@@ -34,5 +34,5 @@
     </collision>
     <collision>
-      <origin xyz="0.6 0.0 0.0" />
+      <origin xyz="-0.5 0.0 0.0" />
       <geometry>
         <sphere radius="0.1" />
