Commit message: Updated kuka launch system and configs for namespace use.

File: agimus_demo_03_mpc_dummy_traj_kuka/urdf/obstacles.xacro (robot description, xacro)
@@ -1,5 +1,4 @@
 <?xml version='1.0' encoding='utf-8'?>
 <robot xmlns:xacro="http://www.ros.org/wiki/xacro" name="pandas">
-    <xacro:include filename="$(find franka_description)/robots/common/utils.xacro" />
     <material name="grey">
         <color rgba=".5 .5 .5 1" />
@@ -21,5 +20,5 @@
         </visual>
     <collision>
-      <origin xyz="0.6 0.0 0.15" />
+      <origin xyz="0.55 0.0 0.25" rpy="0 1.571 0"/>
       <geometry>
         <cylinder length="0.3" radius="0.1" />
@@ -28,5 +27,5 @@
      <!-- Note: these two are deleted in collision model update (robot_model.py)-->
      <collision>
-      <origin xyz="0.6 0.0 0.3" />
+      <origin xyz="0.70 0.0 0.25" />
       <geometry>
         <sphere radius="0.1" />
@@ -34,5 +33,5 @@
     </collision>
     <collision>
-      <origin xyz="0.6 0.0 0.0" />
+      <origin xyz="0.40 0.0 0.25" />
       <geometry>
         <sphere radius="0.1" />

File: agimus_demo_03_mpc_dummy_traj_kuka/urdf/obstacles_none.xacro (robot description, xacro)
@@ -1,5 +1,4 @@
 <?xml version='1.0' encoding='utf-8'?>
 <robot xmlns:xacro="http://www.ros.org/wiki/xacro" name="pandas">
-    <xacro:include filename="$(find franka_description)/robots/common/utils.xacro" />
     <material name="grey">
         <color rgba=".5 .5 .5 1" />
