Commit message: Added run parameter for a tool. Added/updated xacro definitions and models for no tool, sharp tip, and knife.

File: agimus_description/urdf/_materials.urdf.xacro (robot description, xacro)
@@ -10,4 +10,10 @@
       <color rgba="0.5 0.5 0.5 1"/>
     </material>
+    <material name="orange">
+      <color rgba="1.0 0.3 0.0 1"/>
+    </material>
+    <material name="yellow">
+      <color rgba="1.0 0.7 0.0 1"/>
+    </material>
   </xacro:unless>
 </robot>

File: agimus_description/urdf/iiwa7_knife.xacro (robot description, xacro)
@@ -5,5 +5,10 @@
     <!-- include the lbr iiwa description -->
     <xacro:include filename="$(find lbr_description)/urdf/iiwa7/iiwa7.xacro" />
-    <!-- no additional tools -->
+    <!-- include the definition of tools-->
+    <xacro:include filename="$(find agimus_description)/urdf/flange.xacro" />
+    <xacro:include filename="$(find agimus_description)/urdf/knife.xacro" />
+    <!-- connect tools to the end-effector -->
+    <xacro:tool_flange parent="$(arg robot_name)_link_ee" name="$(arg robot_name)_flange"/>
+    <xacro:tool_knife parent="$(arg robot_name)_flange" name="$(arg robot_name)_knife"/>
     <link name="$(arg robot_name)_link_tool">
         <visual>
@@ -16,5 +21,5 @@
     </link>
     <joint name="$(arg robot_name)_joint_tool" type="fixed">
-        <parent link="$(arg robot_name)_link_ee" />
+        <parent link="$(arg robot_name)_knife" />
         <child link="$(arg robot_name)_link_tool" />
         <origin xyz="0 0 0" rpy="0 0 0" />

File: agimus_description/urdf/iiwa7_tip.xacro (robot description, xacro)
@@ -5,5 +5,10 @@
     <!-- include the lbr iiwa description -->
     <xacro:include filename="$(find lbr_description)/urdf/iiwa7/iiwa7.xacro" />
-    <!-- no additional tools -->
+    <!-- include the definition of tools-->
+    <xacro:include filename="$(find agimus_description)/urdf/flange.xacro" />
+    <xacro:include filename="$(find agimus_description)/urdf/sharp_tip.xacro" />
+    <!-- connect tools to the end-effector -->
+    <xacro:tool_flange parent="$(arg robot_name)_link_ee" name="$(arg robot_name)_flange"/>
+    <xacro:tool_sharp_tip parent="$(arg robot_name)_flange" name="$(arg robot_name)_tip"/>
     <link name="$(arg robot_name)_link_tool">
         <visual>
@@ -16,5 +21,5 @@
     </link>
     <joint name="$(arg robot_name)_joint_tool" type="fixed">
-        <parent link="$(arg robot_name)_link_ee" />
+        <parent link="$(arg robot_name)_tip" />
         <child link="$(arg robot_name)_link_tool" />
         <origin xyz="0 0 0" rpy="0 0 0" />
